Commit message: Añadido rplidar al robot

File: turtlebot_uvc_description/urdf/sensors/astra.urdf.xacro (robot description, xacro)
@@ -4,5 +4,4 @@
   <xacro:include filename="$(find turtlebot_uvc_description)/urdf/turtlebot_properties.urdf.xacro"/>
   <!-- Xacro properties -->
-  <xacro:property name="astra_cam_py" value="-0.0125"/>
   <xacro:property name="astra_depth_rel_rgb_py" value="0.0250" />
   <xacro:property name="astra_cam_rel_rgb_py"   value="-0.0125" />
@@ -11,5 +10,5 @@
   <xacro:macro name="sensor_astra" params="parent">
     <joint name="camera_rgb_joint" type="fixed">
-      <origin xyz="${cam_px} ${astra_cam_py} ${cam_pz}"
+      <origin xyz="${cam_px} ${cam_py} ${cam_pz}"
               rpy="0 0 0"/>
       <parent link="${parent}"/>
@@ -31,7 +30,8 @@
     <link name="camera_link">
       <visual>
-        <origin xyz="-0.04 0.02 -0.01" rpy="${M_PI/2} 0 ${M_PI/2}"/>
+        <origin xyz="0 0 0" rpy="${M_PI/2} 0 ${M_PI/2}"/>
         <geometry>
-          <mesh filename="package://turtlebot_description/meshes/sensors/astra.dae" scale="${astra_dae_display_scale} ${astra_dae_display_scale} ${astra_dae_display_scale}"/>
+          <!--mesh filename="package://turtlebot_description/meshes/sensors/astra.dae" scale="${astra_dae_display_scale} ${astra_dae_display_scale} ${astra_dae_display_scale}"/-->
+          <mesh filename="package://turtlebot_uvc_description/meshes/astra2.dae" scale="${astra_dae_display_scale} ${astra_dae_display_scale} ${astra_dae_display_scale}"/>
         </geometry>
       </visual>

File: turtlebot_uvc_description/urdf/turtlebot_common_library.urdf.xacro (robot description, xacro)
@@ -5,5 +5,5 @@
 <robot xmlns:xacro="http://ros.org/wiki/xacro">
   <!-- General -->
-  <xacro:include filename="$(find turtlebot_description)/urdf/common_properties.urdf.xacro"/>
+  <xacro:include filename="$(find turtlebot_uvc_description)/urdf/common_properties.urdf.xacro"/>
   <xacro:include filename="$(find turtlebot_uvc_description)/urdf/turtlebot_properties.urdf.xacro"/>
 </robot>

File: turtlebot_uvc_description/urdf/turtlebot_properties.urdf.xacro (robot description, xacro)
@@ -1,27 +1,9 @@
 <?xml version="1.0"?>
 <robot xmlns:xacro="http://ros.org/wiki/xacro">
-  <!--
-    These properties must be observed by any machine
-    that wants to be defined as a turtlebot. Refer
-    to the REP for more details.
-    http://www.ros.org/reps/rep-0119.html
-   -->
-  <!--
-   ======================================================================
-   - REP 119 : Rgb camera link relative to the Base link
-   ======================================================================
-     Base link is currently defined as the rotational centre on the bottom
-     of the base mould. For both create and kobuki this is actually exactly
-     the same 3d world point.
-     This may cause an issue with a base with much different floor clearance.
-     Should we be using base_footprint for this specification instead?
-     Note: REP needs to be updated with the information below
-     (currently in development and awaiting feedback)
-   -->
+<!--
+  Posicion de la camara RGB-D
+-->
 	<xacro:property name="cam_px" value="-0.087" />
-<!--	<xacro:property name="cam_py" value="-0.0125" /> Y varies for different configurations. get sets in sensors_urdf -->
+	<xacro:property name="cam_py" value="-0.0125" />
 	<xacro:property name="cam_pz" value="0.2870" />
-	<xacro:property name="cam_or" value="0" />
-	<xacro:property name="cam_op" value="0" />
-	<xacro:property name="cam_oy" value="0" />
 </robot>
